File: pcb/timmy.kicad_sch (KiCad schematic)
At the start: 37 parts, among them SW1 SW_Push, SW10 RotaryEncoder_Switch, SW11 RotaryEncoder_Switch, SW2 SW_Push, SW3 SW_Push, SW4 SW_Push, SW5 SW_Push, SW6 SW_Push, SW7 SW_Push, SW8 SW_Push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

Commit message: update to accomodate back-mounted LEDs
Parts:
- D1, D12, D13, D14, D15, D16, D17, D18, D19, D2, D20, D21, D22, D23, D24, D25: footprint LED_SMD:LED_SK6812MINI_PLCC4_3.5x3.5mm_P1.75mm -> libraries:sk6812-mini-e
Changed lines of the file:
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@@
 			)
 		)
-		(property "Footprint" "LED_SMD:LED_SK6812MINI_PLCC4_3.5x3.5mm_P1.75mm"
+		(property "Footprint" "libraries:sk6812-mini-e"
 			(at 340.36 58.42 0)
 			(effects
@@
 			)
 		)
-		(property "Footprint" "LED_SMD:LED_SK6812MINI_PLCC4_3.5x3.5mm_P1.75mm"
+		(property "Footprint" "libraries:sk6812-mini-e"
 			(at 110.49 58.42 0)
 			(effects
@@
 			)
 		)
-		(property "Footprint" "LED_SMD:LED_SK6812MINI_PLCC4_3.5x3.5mm_P1.75mm"
+		(property "Footprint" "libraries:sk6812-mini-e"
 			(at 135.89 58.42 0)
 			(effects
@@
 			)
 		)
-		(property "Footprint" "LED_SMD:LED_SK6812MINI_PLCC4_3.5x3.5mm_P1.75mm"
+		(property "Footprint" "libraries:sk6812-mini-e"
 			(at 161.29 58.42 0)
 			(effects
@@
 			)
 		)
-		(property "Footprint" "LED_SMD:LED_SK6812MINI_PLCC4_3.5x3.5mm_P1.75mm"
+		(property "Footprint" "libraries:sk6812-mini-e"
 			(at 186.69 58.42 0)
 			(effects
@@
 			)
 		)
-		(property "Footprint" "LED_SMD:LED_SK6812MINI_PLCC4_3.5x3.5mm_P1.75mm"
+		(property "Footprint" "libraries:sk6812-mini-e"
 			(at 365.76 58.42 0)
 			(effects
@@
 			)
 		)
-		(property "Footprint" "LED_SMD:LED_SK6812MINI_PLCC4_3.5x3.5mm_P1.75mm"
+		(property "Footprint" "libraries:sk6812-mini-e"
 			(at 262.89 58.42 0)
 			(effects
@@
 			)
 		)
-		(property "Footprint" "LED_SMD:LED_SK6812MINI_PLCC4_3.5x3.5mm_P1.75mm"
+		(property "Footprint" "libraries:sk6812-mini-e"
 			(at 34.29 58.42 0)
 			(effects
@@
 			)
 		)
-		(property "Footprint" "LED_SMD:LED_SK6812MINI_PLCC4_3.5x3.5mm_P1.75mm"
+		(property "Footprint" "libraries:sk6812-mini-e"
 			(at 59.69 58.42 0)
 			(effects
@@
 			)
 		)
-		(property "Footprint" "LED_SMD:LED_SK6812MINI_PLCC4_3.5x3.5mm_P1.75mm"
+		(property "Footprint" "libraries:sk6812-mini-e"
 			(at 314.96 58.42 0)
 			(effects
@@
 			)
 		)
-		(property "Footprint" "LED_SMD:LED_SK6812MINI_PLCC4_3.5x3.5mm_P1.75mm"
+		(property "Footprint" "libraries:sk6812-mini-e"
 			(at 212.09 58.42 0)
 			(effects
@@
 			)
 		)
-		(property "Footprint" "LED_SMD:LED_SK6812MINI_PLCC4_3.5x3.5mm_P1.75mm"
+		(property "Footprint" "libraries:sk6812-mini-e"
 			(at 289.56 58.42 0)
 			(effects
@@
 			)
 		)
-		(property "Footprint" "LED_SMD:LED_SK6812MINI_PLCC4_3.5x3.5mm_P1.75mm"
+		(property "Footprint" "libraries:sk6812-mini-e"
 			(at 391.16 58.42 0)
 			(effects
@@
 			)
 		)
-		(property "Footprint" "LED_SMD:LED_SK6812MINI_PLCC4_3.5x3.5mm_P1.75mm"
+		(property "Footprint" "libraries:sk6812-mini-e"
 			(at 85.09 58.42 0)
 			(effects
@@
 			)
 		)
-		(property "Footprint" "LED_SMD:LED_SK6812MINI_PLCC4_3.5x3.5mm_P1.75mm"
+		(property "Footprint" "libraries:sk6812-mini-e"
 			(at 237.49 58.42 0)
 			(effects
@@
 			)
 		)
-		(property "Footprint" "LED_SMD:LED_SK6812MINI_PLCC4_3.5x3.5mm_P1.75mm"
+		(property "Footprint" "libraries:sk6812-mini-e"
 			(at 416.56 58.42 0)
 			(effects
